Commit message: Update

File: fdplannerw/urdf/robot.urdf.xacro (robot description, xacro)
@@ -100,5 +100,5 @@
     </joint>
     <!-- Wheel macros -->
-    <link name="front_left_wheel">
+    <!-- <link name="front_left_wheel">
         <visual>
             <origin xyz="0 0 0" rpy="0 0 0" />
@@ -167,5 +167,5 @@
         <limit effort="100" velocity="100"/>
         <joint_properties damping="0.0" friction="0.0"/>
-    </joint>
+    </joint> -->
     <!-- Caster macros -->
 	<link name="caster_left_wheel">

File: nbvgplannerw/urdf/robot.urdf.xacro (robot description, xacro)
@@ -100,5 +100,5 @@
     </joint>
     <!-- Wheel macros -->
-    <link name="front_left_wheel">
+    <!-- <link name="front_left_wheel">
         <visual>
             <origin xyz="0 0 0" rpy="0 0 0" />
@@ -167,5 +167,5 @@
         <limit effort="100" velocity="100"/>
         <joint_properties damping="0.0" friction="0.0"/>
-    </joint>
+    </joint> -->
     <!-- Caster macros -->
 	<link name="caster_left_wheel">
